File: NodeMCU-74HC595/hardware/relayboard/relayboard.kicad_pcb (KiCad board)
At the start: 2 copper layers, 43.2 x 39.4 mm, 50 parts, among them J1 Conn_01x01_Male, J10 Conn_01x01_Male, J11 Conn_01x01_Male, J12 Conn_01x01_Male, J13 Conn_01x01_Male, J14 Conn_01x01_Male, J15 Conn_01x01_Male, J16 Conn_01x01_Male, J17 Conn_01x01_Male, J18 Conn_01x01_Male, J19 Conn_01x01_Male, J2 Conn_01x01_Male, J20 Conn_01x01_Male, J21 Conn_01x01_Male, J22 Conn_01x01_Male, J23 Conn_01x01_Male, J24 Conn_01x01_Male, J25 Conn_01x01_Male, J26 Conn_01x01_Male, J27 Conn_01x01_Male, J28 Conn_01x01_Male, J29 Conn_01x01_Male, J3 Conn_01x01_Male, J30 Conn_01x01_Male, J31 Conn_01x01_Male, J32 Conn_01x01_Male, J33 Conn_01x01_Male, J34 Conn_01x01_Male, J35 Conn_01x01_Male, J36 Conn_01x01_Male, J37 Conn_01x01_Male, J38 Conn_01x01_Male, J39 Conn_01x01_Male, J4 Conn_01x01_Male, J40 Conn_01x01_Male, J41 Conn_01x01_Male, J42 Conn_01x01_Male, J43 Conn_01x01_Male, J44 Conn_01x01_Male, J45 Conn_01x01_Male, J46 Conn_01x01_Male, J47 Conn_01x01_Male, J48 Conn_01x01_Male, J49 Conn_01x01_Male, J5 Conn_01x01_Male, J50 Conn_01x01_Male, J6 Conn_01x01_Male, J7 Conn_01x01_Male, J8 Conn_01x01_Male, J9 Conn_01x01_Male

Commit message: fix kicad
Other:
- board text added: "/OE"
- board text added: "/Reset"
- board text added: "3.3V"
- board text added: "5V"
- board text added: "74HC595 Breakout"
- board text added: "Clock"
- board text added: "Data"
- board text added: "Latch"
- board text removed: "+5V"
- board text removed: "SparkFun 74HC595 Breakout"
