File: NodeMCU-74HC595/hardware/mainboard/mainboard.kicad_pcb (KiCad board)
At the start: 2 copper layers, 12 parts, among them J1 Power, J2 Sensor 1, J3 Sensor 2, J4 Display + Buttons, J5 DS3231 RTC, J6 Relay Board, J7 Conn_01x04_Female, U1 Lua-Lolin-v3

Commit message: Update to KiCad 6, improve ReadMe
Other:
- net class Default removed
